File: 04_Electronique/Kicad_Project/LumaDome/LumaDome_Alim/LumaDome_Alim.kicad_sch (KiCad schematic)
At the start: 0 parts

Commit message: Finalisation PCB 02
Parts:
- added H1, H101, H102, H2: MountingHole_Pad, MountingHole:MountingHole_2.2mm_M2_Pad_Via, symbol Mechanical:MountingHole_Pad
- added SW1: SW_SPDT, MaximeRempreinte:B12AV, symbol Switch:SW_SPDT
Connections:
- new net GND: H1.1, H101.1, H102.1, H2.1
- new net Power/Battery_12V: SW1.1 (A)
- new net Power/SW_Sortie: SW1.2 (B)
- new net USBC/Vout: SW1.3 (C)
Other:
- added sheet ESP 32 (ESP_32.kicad_sch)
- added sheet Power (Power.kicad_sch)
- added sheet USBC (USBC.kicad_sch)
- note added: "90 ohm impedance"
- note added: "Choice Source"
- note added: "Fixation"
- note added: "USB connector + ESD connector"
- company: (none) -> ENSEA
- title: (none) -> LumaDome_Alim
