File: 04_Electronique/Kicad_Project/LumaDome/LumaDome_Alim/ESP_32.kicad_sch (KiCad schematic)
At the start: 12 parts, among them J10 Conn_01x04, J7 Conn_02x05_Counter_Clockwise, J8 Conn_01x03, J9 Conn_02x03_Counter_Clockwise, U6 ESP32-WROOM-32E, U7 74AHCT125

Commit message: finalisation PCB
Parts:
- J10: footprint Connector_PinHeader_1.27mm:PinHeader_1x04_P1.27mm_Vertical -> Connector_PinHeader_2.54mm:PinHeader_1x04_P2.54mm_Vertical_SMD_Pin1Left
- J7: footprint Connector_PinHeader_1.27mm:PinHeader_2x05_P1.27mm_Vertical -> Connector_PinHeader_1.27mm:PinHeader_2x05_P1.27mm_Vertical_SMD
- J9: footprint Connector_PinHeader_1.27mm:PinHeader_2x03_P1.27mm_Vertical -> Connector_PinHeader_1.27mm:PinHeader_2x03_P1.27mm_Vertical_SMD
Connections:
- net +5V: now also J8.2 (Pin_2); no longer J8.1 (Pin_1)
- net DIN: now also J8.1 (Pin_1); no longer J8.2 (Pin_2)
Changed lines of the file:
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@@
-	(wire
-		(pts
-			(xy 243.84 64.77) (xy 243.84 66.04)
-		)
-		(stroke
-			(width 0)
-			(type default)
-		)
-	)
 	(wire
 		(pts
@@
 	(wire
 		(pts
-			(xy 243.84 58.42) (xy 243.84 59.69)
-		)
-		(stroke
-			(width 0)
-			(type default)
-		)
-	)
-	(wire
-		(pts
 			(xy 204.47 129.54) (xy 213.36 129.54)
 		)
@@
 	(wire
 		(pts
-			(xy 242.57 62.23) (xy 246.38 62.23)
+			(xy 240.03 62.23) (xy 246.38 62.23)
 		)
 		(stroke
@@
 	(wire
 		(pts
-			(xy 243.84 59.69) (xy 246.38 59.69)
+			(xy 242.57 59.69) (xy 246.38 59.69)
 		)
 		(stroke
@@
 		)
 	)
+	(label "DIN"
+		(at 242.57 59.69 0)
+		(effects
+			(font
+				(size 1.27 1.27)
+			)
+			(justify left bottom)
+		)
+	)
 	(label "Luminosity_button"
 		(at 93.98 83.82 180)
@@
 		)
 	)
-	(label "DIN"
-		(at 242.57 62.23 0)
-		(effects
-			(font
-				(size 1.27 1.27)
-			)
-			(justify left bottom)
-		)
-	)
 	(label "ESP_TDO"
 		(at 85.09 73.66 180)
@@
 	)
 	(symbol
-		(lib_id "power:+5V")
-		(at 243.84 58.42 0)
-		(unit 1)
-		(exclude_from_sim no)
-		(in_bom yes)
-		(on_board yes)
-		(dnp no)
-		(fields_autoplaced yes)
-		(property "Reference" "#PWR049"
-			(at 243.84 62.23 0)
-			(effects
-				(font
-					(size 1.27 1.27)
-				)
-				(hide yes)
-			)
-		)
-		(property "Value" "+5V"
-			(at 243.84 53.34 0)
-			(effects
-				(font
-					(size 1.27 1.27)
-				)
-			)
-		)
-		(property "Footprint" ""
-			(at 243.84 58.42 0)
-			(effects
-				(font
-					(size 1.27 1.27)
-				)
-				(hide yes)
-			)
-		)
-		(property "Datasheet" ""
-			(at 243.84 58.42 0)
-			(effects
-				(font
-					(size 1.27 1.27)
-				)
-				(hide yes)
-			)
-		)
-		(property "Description" "Power symbol creates a global label with name \"+5V\""
-			(at 243.84 58.42 0)
-			(effects
-				(font
-					(size 1.27 1.27)
-				)
-				(hide yes)
-			)
-		)
-		(pin "1"
-		)
-		(instances
-			(project "LumaDome_Alim"
-				(path "/ba8b9c61-a47f-4f27-a45d-48fa5a4c6fc9/87052f3e-4c3f-4ace-a1a5-bfa1bfbc6f4d"
-					(reference "#PWR049")
-					(unit 1)
-				)
-			)
-		)
-	)
-	(symbol
 		(lib_id "power:GND")
 		(at 78.74 36.83 0)
@@
 			)
 		)
-		(property "Footprint" "Connector_PinHeader_1.27mm:PinHeader_2x03_P1.27mm_Vertical"
+		(property "Footprint" "Connector_PinHeader_1.27mm:PinHeader_2x03_P1.27mm_Vertical_SMD"
 			(at 125.73 91.44 0)
 			(effects
@@
 			)
 		)
-		(property "Footprint" "Connector_PinHeader_1.27mm:PinHeader_2x05_P1.27mm_Vertical"
+		(property "Footprint" "Connector_PinHeader_1.27mm:PinHeader_2x05_P1.27mm_Vertical_SMD"
 			(at 123.19 57.15 0)
 			(effects
@@
 	)
 	(symbol
+		(lib_id "power:+5V")
+		(at 240.03 62.23 0)
+		(unit 1)
+		(exclude_from_sim no)
+		(in_bom yes)
+		(on_board yes)
+		(dnp no)
+		(fields_autoplaced yes)
+		(property "Reference" "#PWR037"
+			(at 240.03 66.04 0)
+			(effects
+				(font
+					(size 1.27 1.27)
+				)
+				(hide yes)
+			)
+		)
+		(property "Value" "+5V"
+			(at 240.03 57.15 0)
+			(effects
+				(font
+					(size 1.27 1.27)
+				)
+			)
+		)
+		(property "Footprint" ""
+			(at 240.03 62.23 0)
+			(effects
+				(font
+					(size 1.27 1.27)
+				)
+				(hide yes)
+			)
+		)
+		(property "Datasheet" ""
+			(at 240.03 62.23 0)
+			(effects
+				(font
+					(size 1.27 1.27)
+				)
+				(hide yes)
+			)
+		)
+		(property "Description" "Power symbol creates a global label with name \"+5V\""
+			(at 240.03 62.23 0)
+			(effects
+				(font
+					(size 1.27 1.27)
+				)
+				(hide yes)
+			)
+		)
+		(pin "1"
+		)
+		(instances
+			(project "LumaDome_Alim"
+				(path "/ba8b9c61-a47f-4f27-a45d-48fa5a4c6fc9/87052f3e-4c3f-4ace-a1a5-bfa1bfbc6f4d"
+					(reference "#PWR037")
+					(unit 1)
+				)
+			)
+		)
+	)
+	(symbol
 		(lib_id "power:PWR_FLAG")
 		(at 200.66 147.32 0)
@@
 			)
 		)
-		(property "Footprint" "Connector_PinHeader_1.27mm:PinHeader_1x04_P1.27mm_Vertical"
+		(property "Footprint" "Connector_PinHeader_2.54mm:PinHeader_1x04_P2.54mm_Vertical_SMD_Pin1Left"
 			(at 251.46 31.75 0)
 			(effects
@@
 	(symbol
 		(lib_id "power:GND")
-		(at 243.84 66.04 0)
+		(at 243.84 64.77 0)
 		(unit 1)
 		(exclude_from_sim no)
@@
 		(fields_autoplaced yes)
 		(property "Reference" "#PWR050"
-			(at 243.84 72.39 0)
+			(at 243.84 71.12 0)
 			(effects
 				(font
@@
 		)
 		(property "Value" "GND"
-			(at 243.84 71.12 0)
+			(at 243.84 69.85 0)
 			(effects
 				(font
@@
 		)
 		(property "Footprint" ""
-			(at 243.84 66.04 0)
+			(at 243.84 64.77 0)
 			(effects
 				(font
@@
 		)
 		(property "Datasheet" ""
-			(at 243.84 66.04 0)
+			(at 243.84 64.77 0)
 			(effects
 				(font
@@
 		)
 		(property "Description" "Power symbol creates a global label with name \"GND\" , ground"
-			(at 243.84 66.04 0)
-			(effects
-				(font
+			(at 243.84 64.77 0)
+			(effects
+				(font
