File: 04_Electronique/Kicad_Project/LumaDome/LumaDome_Alim/Power.kicad_sch (KiCad schematic)
At the start: 20 parts, among them J3 Conn_01x02, U3 WE: 173020536, U4 WE: 173010335

Commit message: finalisation PCB
Parts:
- J3: footprint Connector_AMASS:AMASS_XT30U-M_1x02_P5.0mm_Vertical -> Connector_AMASS:AMASS_XT30UPB-F_1x02_P5.0mm_Vertical
Changed lines of the file:
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@@
 			)
 		)
-		(property "Footprint" "Connector_AMASS:AMASS_XT30U-M_1x02_P5.0mm_Vertical"
+		(property "Footprint" "Connector_AMASS:AMASS_XT30UPB-F_1x02_P5.0mm_Vertical"
 			(at 22.86 36.83 0)
 			(effects
